Commit message: Modulo rdf_gazebo con gripper. Invocar con roslaunch rdf_gazebo ur5_bringup.launch gripper:=nombre_de_gripper, actualmente solamente se tiene implementado el robotiq_2f_140, que requiere algunas correcciones para su uso en gazebo

File: catkin_ws/src/dummy_robot_description/urdf/ur5.urdf.xacro (robot description, xacro)
@@ -34,4 +34,5 @@
 				iyy="${0.0833333 * mass * (3 * radius * radius + length * length)}" iyz="0.0"
 				izz="${0.5 * mass * radius * radius}" />
+			<origin xyz="0 0 ${length/2}" rpy="0 0 0"/>
 		</inertial>
 	</xacro:macro>

File: catkin_ws/src/dummy_robot_description/urdf/ur5_gazebo.urdf.xacro (robot description, xacro)
@@ -1,4 +1,4 @@
 <?xml version="1.0"?>
-<robot xmlns:xacro="http://ros.org/wiki/xacro" name="ur5_test" >
+<robot xmlns:xacro="http://ros.org/wiki/xacro" name="ur5_gazebo" >
 	<xacro:arg name="gripper" default="none" />
 	<!-- Arbitrary offsets for shoulder/elbow joints -->
@@ -34,4 +34,5 @@
 				iyy="${0.0833333 * mass * (3 * radius * radius + length * length)}" iyz="0.0"
 				izz="${0.5 * mass * radius * radius}" />
+			<origin xyz="0 0 ${length/2}" rpy="0 0 0"/>
 		</inertial>
 	</xacro:macro>
@@ -47,10 +48,21 @@
 		</visual>
 	</xacro:macro>
+	<xacro:macro name="mesh_collision" params="*origin filename" >
+		<collision>
+ 		   	<xacro:insert_block name="origin"/>
+ 		   	<geometry>
+ 			   	<mesh filename="${filename}"/>
+ 		   	</geometry>
+		</collision>
+   </xacro:macro>
 	<!-- Macro for links -->
 	<!-- Generic link -->
-	<xacro:macro name="generic_link" params="name radius length mass filename *origin">
+	<xacro:macro name="generic_link" params="name radius length mass filename_visual filename_collision *origin">
 		<link name="${name}">
+			<xacro:mesh_collision filename="${filename_collision}">
+				<xacro:insert_block name="origin" />
+			</xacro:mesh_collision>
 			<xacro:inertial_macro radius="${radius}" length="${length}" mass="${mass}"/>
-			<xacro:mesh_visual filename="${filename}">
+			<xacro:mesh_visual filename="${filename_visual}">
 				<xacro:insert_block name="origin" />
 			</xacro:mesh_visual>
@@ -73,26 +85,32 @@
 		</xacro:mesh_visual>
 	</link>
-	<xacro:generic_link name="square_base" radius="${shoulder_radius}" length="${shoulder_height}"
-		mass="${shoulder_mass}" filename="package://ur_description/meshes/ur5/visual/shoulder.dae" >
+	<xacro:generic_link name="square_base" radius="${shoulder_radius}" length="${shoulder_height}" mass="${shoulder_mass}"
+		filename_visual="package://ur_description/meshes/ur5/visual/shoulder.dae"
+		filename_collision="package://ur_description/meshes/ur5/collision/shoulder.stl" >
 		<origin xyz="0 0 0" rpy="0 0 0"/>
 	</xacro:generic_link>
-	<xacro:generic_link name="upper_arm_link" radius="${upper_arm_radius}" length="${upper_arm_length}"
-		mass="${upper_arm_mass}" filename="package://ur_description/meshes/ur5/visual/upperarm.dae" >
+	<xacro:generic_link name="upper_arm_link" radius="${upper_arm_radius}" length="${upper_arm_length}" mass="${upper_arm_mass}"
+		filename_visual="package://ur_description/meshes/ur5/visual/upperarm.dae"
+		filename_collision="package://ur_description/meshes/ur5/collision/upperarm.stl" >
 		<origin xyz="0 0 0" rpy="0 0 0"/>
 	</xacro:generic_link>
-	<xacro:generic_link name="forearm_link" radius="${forearm_radius}" length="${forearm_length}"
-		mass="${forearm_mass}" filename="package://ur_description/meshes/ur5/visual/forearm.dae" >
+	<xacro:generic_link name="forearm_link" radius="${forearm_radius}" length="${forearm_length}" mass="${forearm_mass}"
+		filename_visual="package://ur_description/meshes/ur5/visual/forearm.dae"
+		filename_collision="package://ur_description/meshes/ur5/collision/forearm.stl" >
 		<origin xyz="0 0 0" rpy="0 0 0"/>
 	</xacro:generic_link>
-	<xacro:generic_link name="wrist_1_link" radius="${wrist_radius}" length="${wrist_1_length}"
-		mass="${wrist_1_mass}" filename="package://ur_description/meshes/ur5/visual/wrist1.dae" >
+	<xacro:generic_link name="wrist_1_link" radius="${wrist_radius}" length="${wrist_1_length}"	mass="${wrist_1_mass}"
+		filename_visual="package://ur_description/meshes/ur5/visual/wrist1.dae"
+		filename_collision="package://ur_description/meshes/ur5/collision/wrist1.stl" >
 		<origin xyz="0 0 0" rpy="0 0 0"/>
 	</xacro:generic_link>
-	<xacro:generic_link name="wrist_2_link" radius="${wrist_radius}" length="${wrist_2_length}"
-		mass="${wrist_2_mass}" filename="package://ur_description/meshes/ur5/visual/wrist2.dae" >
+	<xacro:generic_link name="wrist_2_link" radius="${wrist_radius}" length="${wrist_2_length}"	mass="${wrist_2_mass}"
+		filename_visual="package://ur_description/meshes/ur5/visual/wrist2.dae"
+		filename_collision="package://ur_description/meshes/ur5/collision/wrist2.stl" >
 		<origin xyz="0 0 0" rpy="0 0 0"/>
 	</xacro:generic_link>
-	<xacro:generic_link name="wrist_3_link" radius="${wrist_radius}" length="${wrist_3_length}"
-		mass="${wrist_3_mass}" filename="package://ur_description/meshes/ur5/visual/wrist3.dae" >
+	<xacro:generic_link name="wrist_3_link" radius="${wrist_radius}" length="${wrist_3_length}"	mass="${wrist_3_mass}"
+		filename_visual="package://ur_description/meshes/ur5/visual/wrist3.dae"
+		filename_collision="package://ur_description/meshes/ur5/collision/wrist3.stl" >
 		<origin xyz="0 0 0" rpy="0 0 0"/>
 	</xacro:generic_link>
@@ -131,3 +149,33 @@
 		</joint>
 	</xacro:if>
+	<!-- Gazebo -->
+	<gazebo reference="square_base">
+ 		<mu1>0.2</mu1>
+    	<mu2>0.2</mu2>
+  	</gazebo>
+	<gazebo reference="upper_arm_link">
+ 		<mu1>0.2</mu1>
+    	<mu2>0.2</mu2>
+  	</gazebo>
+	<gazebo reference="forearm_link">
+ 		<mu1>0.2</mu1>
+    	<mu2>0.2</mu2>
+  	</gazebo>
+	<gazebo reference="wrist_1_link">
+ 		<mu1>0.2</mu1>
+    	<mu2>0.2</mu2>
+  	</gazebo>
+	<gazebo reference="wrist_2_link">
+ 		<mu1>0.2</mu1>
+    	<mu2>0.2</mu2>
+  	</gazebo>
+	<gazebo reference="wrist_3_link">
+ 		<mu1>0.2</mu1>
+    	<mu2>0.2</mu2>
+  	</gazebo>
+	<link name="world" />
+	<joint name="fixed" type="fixed">
+    	<parent link="world"/>
+    	<child link="base_link"/>
+  	</joint>
 </robot>
