Commit message: Se incluyen ultimas practicas

File: catkin_ws_old/src/ur5_gripper_description/urdf/ur5_gripper.urdf (robot description, URDF)
Before this commit: robot ur5_gripper, 22 links, 21 joints
Links:
- removed link vacuum_gripper
Joints:
- removed joint gripper_joint

File: catkin_ws_old/src/ur5_gripper_description/urdf/ur5_gripper.urdf.xacro (robot description, xacro)
@@ -11,22 +11,6 @@
 	</joint>
     <xacro:robotiq_85_gripper prefix="" parent="tool0" >
-	    <origin xyz="0 0 0" rpy="0 -1.57 0"/>
+	    <origin xyz="0 0 0" rpy="0 -1.57079 0"/>
     </xacro:robotiq_85_gripper>
-    <link name="vacuum_gripper">
-      <gravity>0</gravity>
-      <inertial>
-        <origin rpy="0 0.050 0" xyz="0.000000 0.000000 0.000000"/>
-        <mass value="0.0001"/>
-        <inertia ixx="1e-08" ixy="0" ixz="0" iyy="1e-08" iyz="0" izz="1e-08"/>
-      </inertial>
-    </link>
-         <joint name="gripper_joint" type="revolute">
-      <axis xyz="1 0 0" />
-      <parent link="tool0" />
-      <child link="vacuum_gripper" />
-      <origin rpy="0 0 0" xyz="0.0 0.0 0.14" />
-      <limit effort="50" velocity="50" lower="0" upper="0" />
-      <dynamics damping="0.0" friction="10"/>
-    </joint>
     <gazebo reference="shoulder_link">
       <selfCollide>true</selfCollide>
@@ -47,19 +31,11 @@
       <selfCollide>true</selfCollide>
     </gazebo>
-    <gazebo reference="tool0">
+    <gazebo reference="ee_link">
       <selfCollide>true</selfCollide>
     </gazebo>
-       <gazebo>
+    <gazebo>
       <plugin name="ros_control" filename="libgazebo_ros_control.so">
         <!--robotNamespace>/</robotNamespace-->
         <!--robotSimType>gazebo_ros_control/DefaultRobotHWSim</robotSimType-->
-      </plugin>
-           <plugin name="gazebo_ros_vacuum_gripper" filename="libgazebo_ros_vacuum_gripper.so">
-        <robotNamespace>/ur5/vacuum_gripper</robotNamespace>
-        <bodyName>vacuum_gripper</bodyName>
-        <topicName>grasping</topicName>
-	<maxForce>10</maxForce>
-        <maxDistance>0.05</maxDistance>
-        <minDistance>0.01</minDistance>
       </plugin>
    <plugin name="gazebo_grasp_fix" filename="libgazebo_grasp_fix.so">
@@ -72,9 +48,9 @@
         </arm>
       <forces_angle_tolerance>100</forces_angle_tolerance>
-      <update_rate>20</update_rate>
-      <grip_count_threshold>4</grip_count_threshold>
+      <update_rate>4</update_rate>
+      <grip_count_threshold>1</grip_count_threshold>
       <max_grip_count>8</max_grip_count>
-      <release_tolerance>0.00091</release_tolerance>
-      <disable_collisions_on_attach>true</disable_collisions_on_attach>
+      <release_tolerance>0.015</release_tolerance>
+      <disable_collisions_on_attach>false</disable_collisions_on_attach>
       <contact_topic>__default_topic__</contact_topic>
     </plugin>
